File: pcb/Quatro.kicad_sch (KiCad schematic)
At the start: 98 parts, among them J1 BATTERY, J2 BATTERY, J3 Conn_01x02, J4 UART1 SH, J5 st-link SH, J6 2.54mm 02x03, J7 2.54mm 02x03, Q1 IRLML6402, Q2 IRFML8244, Q3 BSS138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

Commit message: pcb作成して発注
Parts:
- U8, U9: footprint My_Device:DRV8835 -> Quatro:DRV8835
Changed lines of the file:
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@@
     (property "Reference" "U8" (id 0) (at 365.76 144.78 0))
     (property "Value" "DRV8835" (id 1) (at 365.76 147.32 0))
-    (property "Footprint" "My_Device:DRV8835" (id 2) (at 350.52 142.24 0)
+    (property "Footprint" "Quatro:DRV8835" (id 2) (at 350.52 142.24 0)
       (effects (font (size 1.27 1.27)) hide)
     )
@@
     (property "Reference" "U9" (id 0) (at 365.76 194.31 0))
     (property "Value" "DRV8835" (id 1) (at 365.76 196.85 0))
-    (property "Footprint" "My_Device:DRV8835" (id 2) (at 350.52 191.77 0)
+    (property "Footprint" "Quatro:DRV8835" (id 2) (at 350.52 191.77 0)
       (effects (font (size 1.27 1.27)) hide)
     )
@@
     )
     (path "/00000000-0000-0000-0000-000060d47ace"
-      (reference "U8") (unit 1) (value "DRV8835") (footprint "My_Device:DRV8835")
+      (reference "U8") (unit 1) (value "DRV8835") (footprint "Quatro:DRV8835")
     )
     (path "/00000000-0000-0000-0000-000060ed4ff2"
-      (reference "U9") (unit 1) (value "DRV8835") (footprint "My_Device:DRV8835")
+      (reference "U9") (unit 1) (value "DRV8835") (footprint "Quatro:DRV8835")
     )
   )
